File: main.sch (EAGLE design)
At the start: 14 parts, among them IC1 TL071P

Commit message: Convert to smd.
Parts:
- removed IN-, OUT-: (no value), wirepad:2,54/0,8
- added GND: WIREPAD2,15/1,0, wirepad:WIREPAD2,15/1,0
- C1, C2: device rcl:CPOL-USE2.5-5 -> rcl:CPOL-USB
- C3: device rcl:C-US050-025X075 -> rcl:C-USC0805
- IN, OUT, V+: value (none) -> WIREPAD2,15/1,0; device wirepad:2,54/0,8 -> wirepad:WIREPAD2,15/1,0
- R1, R2, R3, R4, R5: device resistor:R-US_0204/7 -> rcl:R-US_R0805
Connections:
- net GND: now also GND.P; no longer IN-.P, OUT-.P
Changed lines of the file:
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@@
 <?xml version="1.0" encoding="utf-8"?>
 <!DOCTYPE eagle SYSTEM "eagle.dtd">
-<eagle version="8.0.2">
+<eagle version="8.1.0">
 <drawing>
 <settings>
@@
 <grid distance="0.1" unitdist="inch" unit="inch" style="lines" multiple="1" display="no" altdistance="0.01" altunitdist="inch" altunit="inch"/>
 <layers>
-<layer number="1" name="Top" color="4" fill="1" visible="no" active="no"/>
-<layer number="16" name="Bottom" color="1" fill="1" visible="no" active="no"/>
-<layer number="17" name="Pads" color="2" fill="1" visible="no" active="no"/>
-<layer number="18" name="Vias" color="2" fill="1" visible="no" active="no"/>
-<layer number="19" name="Unrouted" color="6" fill="1" visible="no" active="no"/>
-<layer number="20" name="Dimension" color="15" fill="1" visible="no" active="no"/>
-<layer number="21" name="tPlace" color="7" fill="1" visible="no" active="no"/>
-<layer number="22" name="bPlace" color="7" fill="1" visible="no" active="no"/>
-<layer number="23" name="tOrigins" color="15" fill="1" visible="no" active="no"/>
-<layer number="24" name="bOrigins" color="15" fill="1" visible="no" active="no"/>
-<layer number="25" name="tNames" color="7" fill="1" visible="no" active="no"/>
-<layer number="26" name="bNames" color="7" fill="1" visible="no" active="no"/>
-<layer number="27" name="tValues" color="7" fill="1" visible="no" active="no"/>
-<layer number="28" name="bValues" color="7" fill="1" visible="no" active="no"/>
+<layer number="1" name="Top" color="4" fill="1" visible="yes" active="no"/>
+<layer number="16" name="Bottom" color="1" fill="1" visible="yes" active="no"/>
+<layer number="17" name="Pads" color="2" fill="1" visible="yes" active="no"/>
+<layer number="18" name="Vias" color="2" fill="1" visible="yes" active="no"/>
+<layer number="19" name="Unrouted" color="6" fill="1" visible="yes" active="no"/>
+<layer number="20" name="Dimension" color="15" fill="1" visible="yes" active="no"/>
+<layer number="21" name="tPlace" color="7" fill="1" visible="yes" active="no"/>
+<layer number="22" name="bPlace" color="7" fill="1" visible="yes" active="no"/>
+<layer number="23" name="tOrigins" color="15" fill="1" visible="yes" active="no"/>
+<layer number="24" name="bOrigins" color="15" fill="1" visible="yes" active="no"/>
+<layer number="25" name="tNames" color="7" fill="1" visible="yes" active="no"/>
+<layer number="26" name="bNames" color="7" fill="1" visible="yes" active="no"/>
+<layer number="27" name="tValues" color="7" fill="1" visible="yes" active="no"/>
+<layer number="28" name="bValues" color="7" fill="1" visible="yes" active="no"/>
 <layer number="29" name="tStop" color="7" fill="3" visible="no" active="no"/>
 <layer number="30" name="bStop" color="7" fill="6" visible="no" active="no"/>
@@
 <layer number="35" name="tGlue" color="7" fill="4" visible="no" active="no"/>
 <layer number="36" name="bGlue" color="7" fill="5" visible="no" active="no"/>
-<layer number="37" name="tTest" color="7" fill="1" visible="no" active="no"/>
-<layer number="38" name="bTest" color="7" fill="1" visible="no" active="no"/>
+<layer number="37" name="tTest" color="7" fill="1" visible="yes" active="no"/>
+<layer number="38" name="bTest" color="7" fill="1" visible="yes" active="no"/>
 <layer number="39" name="tKeepout" color="4" fill="11" visible="no" active="no"/>
 <layer number="40" name="bKeepout" color="1" fill="11" visible="no" active="no"/>
@@
 <layer number="44" name="Drills" color="7" fill="1" visible="no" active="no"/>
 <layer number="45" name="Holes" color="7" fill="1" visible="no" active="no"/>
-<layer number="46" name="Milling" color="3" fill="1" visible="no" active="no"/>
-<layer number="47" name="Measures" color="7" fill="1" visible="no" active="no"/>
-<layer number="48" name="Document" color="7" fill="1" visible="no" active="no"/>
-<layer number="49" name="Reference" color="7" fill="1" visible="no" active="no"/>
-<layer number="51" name="tDocu" color="7" fill="1" visible="no" active="no"/>
-<layer number="52" name="bDocu" color="7" fill="1" visible="no" active="no"/>
+<layer number="46" name="Milling" color="3" fill="1" visible="yes" active="no"/>
+<layer number="47" name="Measures" color="7" fill="1" visible="yes" active="no"/>
+<layer number="48" name="Document" color="7" fill="1" visible="yes" active="no"/>
+<layer number="49" name="Reference" color="7" fill="1" visible="yes" active="no"/>
+<layer number="51" name="tDocu" color="7" fill="1" visible="yes" active="no"/>
+<layer number="52" name="bDocu" color="7" fill="1" visible="yes" active="no"/>
 <layer number="90" name="Modules" color="5" fill="1" visible="yes" active="yes"/>
 <layer number="91" name="Nets" color="2" fill="1" visible="yes" active="yes"/>
@@
 </classes>
 <parts>
-<part name="R1" library="resistor" deviceset="R-US_" device="0204/7" value="1M"/>
-<part name="R2" library="resistor" deviceset="R-US_" device="0204/7" value="1M"/>
-<part name="R3" library="resistor" deviceset="R-US_" device="0204/7" value="1M"/>
-<part name="R4" library="resistor" deviceset="R-US_" device="0204/7" value="100k"/>
-<part name="R5" library="resistor" deviceset="R-US_" device="0204/7" value="220k"/>
-<part name="C1" library="rcl" deviceset="CPOL-US" device="E2.5-5" value="10u"/>
-<part name="C2" library="rcl" deviceset="CPOL-US" device="E2.5-5" value="10uf"/>
-<part name="C3" library="rcl" deviceset="C-US" device="050-025X075" value="100n"/>
-<part name="IC1" library="linear" deviceset="TL071" device="P"/>
+<part name="R1" library="rcl" deviceset="R-US_" device="R0805" value="1M"/>
+<part name="R2" library="rcl" deviceset="R-US_" device="R0805" value="1M"/>
+<part name="R3" library="rcl" deviceset="R-US_" device="R0805" value="1M"/>
+<part name="R4" library="rcl" deviceset="R-US_" device="R0805" value="100k"/>
+<part name="R5" library="rcl" deviceset="R-US_" device="R0805" value="220k"/>
+<part name="C1" library="rcl" deviceset="CPOL-US" device="B" value="10u"/>
+<part name="C2" library="rcl" deviceset="CPOL-US" device="B" value="10uf"/>
+<part name="C3" library="rcl" deviceset="C-US" device="C0805" value="100n"/>
+<part name="IC1" library="linear" deviceset="TL071" device="P" value="TL071P"/>
 <part name="SUPPLY1" library="supply2" deviceset="GND" device=""/>
 <part name="SUPPLY2" library="supply2" deviceset="GND" device=""/>
 <part name="SUPPLY3" library="supply2" deviceset="GND" device=""/>
-<part name="IN" library="wirepad" deviceset="2,54/0,8" device=""/>
-<part name="IN-" library="wirepad" deviceset="2,54/0,8" device=""/>
-<part name="OUT" library="wirepad" deviceset="2,54/0,8" device=""/>
-<part name="OUT-" library="wirepad" deviceset="2,54/0,8" device=""/>
+<part name="IN" library="wirepad" deviceset="WIREPAD" device="2,15/1,0"/>
+<part name="GND" library="wirepad" deviceset="WIREPAD" device="2,15/1,0"/>
+<part name="OUT" library="wirepad" deviceset="WIREPAD" device="2,15/1,0"/>
 <part name="SUPPLY5" library="supply2" deviceset="GND" device=""/>
-<part name="SUPPLY6" library="supply2" deviceset="GND" device=""/>
-<part name="V+" library="wirepad" deviceset="2,54/0,8" device=""/>
+<part name="V+" library="wirepad" deviceset="WIREPAD" device="2,15/1,0"/>
 </parts>
 <sheets>
@@
 <instance part="SUPPLY2" gate="GND" x="33.02" y="30.48"/>
 <instance part="SUPPLY3" gate="GND" x="63.5" y="43.18"/>
-<instance part="IN" gate="P" x="-5.08" y="55.88"/>
-<instance part="IN-" gate="P" x="-5.08" y="45.72"/>
-<instance part="OUT" gate="P" x="99.06" y="53.34" rot="R180"/>
-<instance part="OUT-" gate="P" x="99.06" y="43.18" rot="R180"/>
-<instance part="SUPPLY5" gate="GND" x="2.54" y="38.1"/>
-<instance part="SUPPLY6" gate="GND" x="91.44" y="35.56"/>
-<instance part="V+" gate="P" x="33.02" y="81.28" rot="R270"/>
+<instance part="IN" gate="G$1" x="-5.08" y="55.88"/>
+<instance part="GND" gate="G$1" x="20.32" y="81.28" rot="R270"/>
+<instance part="OUT" gate="G$1" x="99.06" y="53.34" rot="R180"/>
+<instance part="SUPPLY5" gate="GND" x="20.32" y="68.58"/>
+<instance part="V+" gate="G$1" x="33.02" y="81.28" rot="R270"/>
 </instances>
 <busses>
@@
 <pinref part="C3" gate="G$1" pin="1"/>
 <wire x1="12.7" y1="55.88" x2="20.32" y2="55.88" width="0.1524" layer="91"/>
-<pinref part="IN" gate="P" pin="P"/>
+<pinref part="IN" gate="G$1" pin="P"/>
 <wire x1="-2.54" y1="55.88" x2="12.7" y2="55.88" width="0.1524" layer="91"/>
 <junction x="12.7" y="55.88"/>
@@
 </segment>
 <segment>
-<pinref part="IN-" gate="P" pin="P"/>
+<pinref part="GND" gate="G$1" pin="P"/>
 <pinref part="SUPPLY5" gate="GND" pin="GND"/>
-<wire x1="-2.54" y1="45.72" x2="2.54" y2="45.72" width="0.1524" layer="91"/>
-<wire x1="2.54" y1="45.72" x2="2.54" y2="40.64" width="0.1524" layer="91"/>
-</segment>
-<segment>
-<pinref part="OUT-" gate="P" pin="P"/>
-<pinref part="SUPPLY6" gate="GND" pin="GND"/>
-<wire x1="96.52" y1="43.18" x2="91.44" y2="43.18" width="0.1524" layer="91"/>
-<wire x1="91.44" y1="43.18" x2="91.44" y2="38.1" width="0.1524" layer="91"/>
+<wire x1="20.32" y1="78.74" x2="20.32" y2="71.12" width="0.1524" layer="91"/>
 </segment>
 </net>
@@
 <segment>
 <pinref part="C2" gate="G$1" pin="-"/>
-<pinref part="OUT" gate="P" pin="P"/>
+<pinref part="OUT" gate="G$1" pin="P"/>
 <wire x1="91.44" y1="53.34" x2="96.52" y2="53.34" width="0.1524" layer="91"/>
 </segment>
@@
 <wire x1="33.02" y1="73.66" x2="33.02" y2="78.74" width="0.1524" layer="91"/>
 <junction x="33.02" y="73.66"/>
-<pinref part="V+" gate="P" pin="P"/>
-</segment>
-</net>
+<pinref part="V+" gate="G$1" pin="P"/>
+</segment>
+</net>

Commit message: Add more clearance between cap and a dip socket.
Parts:
- C1, C2: device rcl:CPOL-USB -> rcl:CPOL-USC
Changed lines of the file:
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@@
 <part name="R4" library="rcl" deviceset="R-US_" device="R0805" value="100k"/>
 <part name="R5" library="rcl" deviceset="R-US_" device="R0805" value="220k"/>
-<part name="C1" library="rcl" deviceset="CPOL-US" device="B" value="10u"/>
-<part name="C2" library="rcl" deviceset="CPOL-US" device="B" value="10uf"/>
+<part name="C1" library="rcl" deviceset="CPOL-US" device="C" value="10u"/>
+<part name="C2" library="rcl" deviceset="CPOL-US" device="C" value="10uf"/>
 <part name="C3" library="rcl" deviceset="C-US" device="C0805" value="100n"/>
 <part name="IC1" library="linear" deviceset="TL071" device="P" value="TL071P"/>
